File: kicad/state-variable-filter.kicad_pcb (KiCad board)
At the start: 2 copper layers, 99 x 110 mm, 113 parts, among them J1 AudioJack2_SwitchT, J10 AudioJack2_SwitchT, J11 AudioJack2_SwitchT, J12 Conn_01x08_Pin, J13 Conn_01x08_Socket, J14 Conn_01x08_Pin, J15 Conn_02x05_Odd_Even, J2 Conn_01x08_Socket, J3 AudioJack2_SwitchT, J4 AudioJack2_SwitchT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

Commit message: Fixing minor BOM value issues
Parts:
- C9: value 20pF -> 22pF
- RV2, RV3, RV6: value 10k -> 10kB
Changed lines of the file:
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@@
 			)
 		)
-		(property "Value" "10k"
+		(property "Value" "10kB"
 			(at 0 10.795 180)
 			(layer "F.Fab")
@@
 			)
 		)
-		(property "Value" "10k"
+		(property "Value" "10kB"
 			(at 0 10.795 180)
 			(layer "F.Fab")
@@
 			)
 		)
-		(property "Value" "10k"
+		(property "Value" "10kB"
 			(at 0 10.795 180)
 			(layer "F.Fab")
@@
 			)
 		)
-		(property "Value" "20pF"
+		(property "Value" "22pF"
 			(at 2.5 0 0)
 			(layer "F.Fab")

Commit message: Updating schematic after value tweaks
and regenerating BOMs
Parts:
- D12, D3, D4: value 1n4148 -> 1N4148
- R12: value 100k -> 270k
- R33: value 100k -> 150k
- R7: value 180k -> 100k
- R8: value 1M5 -> 1m5
Changed lines of the file:
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@@
 			)
 		)
-		(property "Value" "1M5"
+		(property "Value" "1m5"
 			(at 8.128 0.6 0)
 			(layer "F.Fab")
@@
 			)
 		)
-		(property "Value" "1n4148"
+		(property "Value" "1N4148"
 			(at 3.81 0 0)
 			(layer "F.Fab")
@@
 		(sheetname "/")
 		(sheetfile "state-variable-filter.kicad_sch")
-		(attr through_hole)
+		(attr through_hole dnp)
 		(fp_line
 			(start 6.58 0)
@@
 		(sheetname "/")
 		(sheetfile "state-variable-filter.kicad_sch")
-		(attr through_hole)
+		(attr through_hole dnp)
 		(fp_line
 			(start 8.35 -1.37)
@@
 			)
 		)
-		(property "Value" "1n4148"
+		(property "Value" "1N4148"
 			(at 3.81 0.032 0)
 			(layer "F.Fab")
@@
 		(sheetname "/")
 		(sheetfile "state-variable-filter.kicad_sch")
-		(attr through_hole)
+		(attr through_hole dnp)
 		(fp_line
 			(start 9.12 0)
@@
 			)
 		)
-		(property "Value" "1n4148"
+		(property "Value" "1N4148"
 			(at 3.81 0 0)
 			(layer "F.Fab")
@@
 			)
 		)
-		(property "Value" "100k"
+		(property "Value" "270k"
 			(at 8.128 0.6 0)
 			(layer "F.Fab")
@@
 			)
 		)
-		(property "Value" "100k"
+		(property "Value" "150k"
 			(at 8.128 0.6 90)
 			(layer "F.Fab")
@@
 		(sheetname "/")
 		(sheetfile "state-variable-filter.kicad_sch")
-		(attr through_hole)
+		(attr through_hole dnp)
 		(fp_line
 			(start 9.12 0)
@@
 			)
 		)
-		(property "Spec" "ceramic C0G"
+		(property "Spec" "ceramic X7R"
 			(at 0 0 0)
 			(unlocked yes)
@@
 			)
 		)
-		(property "Value" "180k"
+		(property "Value" "100k"
 			(at 8.128 0.6 90)
 			(layer "F.Fab")
@@
 		(sheetname "/")
 		(sheetfile "state-variable-filter.kicad_sch")
-		(attr through_hole)
+		(attr through_hole exclude_from_bom)
 		(fp_circle
 			(center 0 0)
@@
 		(sheetname "/")
 		(sheetfile "state-variable-filter.kicad_sch")
-		(attr through_hole)
+		(attr through_hole exclude_from_bom)
 		(fp_circle
 			(center 0 0)
@@
 		(sheetname "/")
 		(sheetfile "state-variable-filter.kicad_sch")
-		(attr through_hole)
+		(attr through_hole exclude_from_bom)
 		(fp_circle
 			(center 0 0)
@@
 			)
 		)
+		(property "Spec" "aluminium electrolytic"
+			(at 0 0 0)
+			(unlocked yes)
+			(layer "B.Fab")
+			(hide yes)
+			(effects
+				(font
+					(size 1 1)
+					(thickness 0.15)
+				)
+				(justify mirror)
+			)
+		)
 		(property ki_fp_filters "CP_*")
 		(sheetname "/")
@@
 		(sheetname "/")
 		(sheetfile "state-variable-filter.kicad_sch")
-		(attr through_hole)
+		(attr through_hole dnp)
 		(fp_line
 			(start 1.38 -1.27)
@@
 		(sheetname "/")
 		(sheetfile "state-variable-filter.kicad_sch")
-		(attr through_hole)
+		(attr through_hole exclude_from_bom)
 		(fp_circle
 			(center 0 0)
@@
 		(sheetname "/")
 		(sheetfile "state-variable-filter.kicad_sch")
-		(attr through_hole)
+		(attr through_hole dnp)
 		(fp_line
 			(start -1.38 -3.92)
@@
 			)
 		)
+		(property "Spec" "aluminium electrolytic"
+			(at 0 0 0)
+			(unlocked yes)
+			(layer "B.Fab")
+			(hide yes)
+			(effects
+				(font
+					(size 1 1)
+					(thickness 0.15)
+				)
+				(justify mirror)
+			)
+		)
 		(property ki_fp_filters "CP_*")
 		(sheetname "/")
@@
 		(sheetname "/")
 		(sheetfile "state-variable-filter.kicad_sch")
-		(attr through_hole)
+		(attr through_hole dnp)
 		(fp_line
 			(start -1.38 1.38)

Commit message: Updating with rev02 fixes
Parts:
- added C21: 5pF, Rumblesan_Standard_Parts:C_Rect_L7.0mm_W2.5mm_P5.00mm, F.Cu at (162.9, 108.6)
- added C22: 5pF, Rumblesan_Standard_Parts:C_Rect_L7.0mm_W2.5mm_P5.00mm, F.Cu at (162.8, 103.2)
- added R38: 47k, Rumblesan_Standard_Parts:R_Axial_DIN0207_L6.3mm_D2.5mm_P10.16mm_Horizontal, F.Cu at (124.1, 97.5)
- moved JP1 3.14 mm to (157.5, 87.8)
- moved R19 3.05 mm to (165.9, 66.5)
- moved R35 3.05 mm to (162.8, 66.5)
- moved C15 1.97 mm to (161.0, 95.1)
- moved JP2 1.65 mm to (132.7, 120.7)
- moved R11 1.53 mm to (137.2, 96.6)
- moved R15 1.40 mm to (135.5, 114.3)
- moved C7 1.40 mm to (135.8, 117.1)
- moved C6 1.35 mm to (130.8, 100.1)
- moved C5 1.27 mm to (132.6, 104.4)
- moved U3 1.27 mm to (146.8, 117.9)
- moved C13 1.15 mm to (151.3, 84.2)
- moved C17 1.14 mm to (159.9, 114.8)
- moved D7 1.14 mm to (160.1, 105.9)
- moved D8 1.14 mm to (157.6, 96.5)
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Connections:
- J1 pad TN: GND -> unconnected-(J1-PadTN)
- J5 pad TN: GND -> unconnected-(J5-PadTN)
- J6 pad TN: GND -> unconnected-(J6-PadTN)
- J7 pad TN: GND -> unconnected-(J7-PadTN)
Routing:
- net Net-(D7-A): track 11.7 -> 27.5 mm
- net Net-(C22-Pad2): track 6.31 -> 20.0 mm
- net HI_PASS_OUTPUT: track 76.0 -> 79.4 mm
- net Net-(C15-Pad1): track 3.15 -> 5.32 mm
- net FREQ_VC: track 29.2 -> 31.0 mm, vias 0 -> 1
- net Net-(U2D--): track 30.0 -> 28.3 mm
- net Net-(JP2-B): track 4.13 -> 5.78 mm
- net Net-(JP1-A): track 10.2 -> 11.8 mm
- net Net-(R11-Pad1): track 28.7 -> 27.2 mm
- net /PING_MAIN: track 49.1 -> 50.6 mm
- net /FILTER_INPUT_1_MAIN: track 25.8 -> 26.9 mm
- net VCC: track 142.2 -> 143.1 mm
- net Net-(U2A--): track 35.8 -> 36.7 mm
- net RES_VC: track 50.3 -> 49.7 mm
- net /RES_ATTV_CW_MAIN: track 52.6 -> 53.2 mm
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Other:
- board text added: "BCM SVF ${REVISION}"
